Commit message: feat(puzzlebot_description): add ament_cmake package for robot model
Move URDF, STL meshes, and RViz config out of the monolithic
puzzlebot_sim package into a dedicated puzzlebot_description package.
Update all mesh references from package://puzzlebot_sim to
package://puzzlebot_description.

Co-Authored-By: Claude Sonnet 4.6 <noreply@anthropic.com>

File: src/puzzlebot_description/urdf/puzzlebot.urdf (robot description, URDF)
Before this commit: robot Puzzlebot_Jetson_Lidar_Ed., 5 links, 4 joints
Links:
- link base_link: geometry visual mesh filename=package://puzzlebot_description/meshes/Puzzlebot_Jetson_Lid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
- link caster_link: geometry visual mesh filename=package://puzzlebot_description/meshes/Puzzlebot_Caster_Whe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
- link wheel_l_link: geometry visual mesh filename=package://puzzlebot_description/meshes/Puzzlebot_Wheel.stl
- link wheel_r_link: geometry visual mesh filename=package://puzzlebot_description/meshes/Puzzlebot_Wheel.stl

Commit message: feat(description): add collision, inertia, Gazebo plugins, lidar and camera sensors to URDF
- Add collision geometry and inertial properties to base_link and wheels
- Add differential drive plugin (libgazebo_ros_diff_drive)
- Add 360° LiDAR sensor publishing /scan (LaserScan)
- Add camera sensor publishing /cam_img and /cam_info
- Update RViz config to display lidar_link and /map topic

Co-Authored-By: Claude Sonnet 4.6 <noreply@anthropic.com>

File: src/puzzlebot_description/urdf/puzzlebot.urdf (robot description, URDF)
Before this commit: robot Puzzlebot_Jetson_Lidar_Ed., 5 links, 4 joints
Links:
- added link lidar_link, mass 0.1; collision cylinder length=0.04 radius=0.04; visual cylinder length=0.04 radius=0.04
- link base_link: mass None -> 2.0; geometry collision box size=0.20 0.15 0.10; visual mesh filename=package://puzzlebot_description/meshes/Puzzlebot_Jetson_Lid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
- link caster_link: mass None -> 0.05; geometry collision sphere radius=0.02; visual mesh filename=package://puzzlebot_description/meshes/Puzzlebot_Caster_Whe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
- link wheel_l_link: mass None -> 0.2; geometry collision cylinder length=0.03 radius=0.05; visual mesh filename=package://puzzlebot_description/meshes/Puzzlebot_Wheel.stl
- link wheel_r_link: mass None -> 0.2; geometry collision cylinder length=0.03 radius=0.05; visual mesh filename=package://puzzlebot_description/meshes/Puzzlebot_Wheel.stl
Joints:
- added joint lidar_joint: type fixed, parent base_link, child lidar_link, origin xyz=0.0 0.0 0.15 rpy=0 0 0
