Commit message: chore: Last Slam

File: src/puzzlebot_description/urdf/puzzlebot_gz.urdf (robot description, URDF)
Before this commit: robot puzzlebot, 6 links, 5 joints
Links:
- added link camera_link, mass 0.05; visual box size=0.025 0.090 0.025
Joints:
- added joint camera_joint: type fixed, parent base_link, child camera_link, origin xyz=0.152 0.000 0.044 rpy=0 0 0

Commit message: commit last slam commit

File: src/puzzlebot_description/urdf/puzzlebot_gz.urdf (robot description, URDF)
Before this commit: robot puzzlebot, 7 links, 6 joints
Joints:
- joint lidar_joint: origin xyz=0.0 0.0 0.15 rpy=0 0 0 -> xyz=0.0 0.0 0.175 rpy=0 0 0
